File: pip-kicad/pip-kicad.kicad_sch (KiCad schematic)
At the start: 6 parts, among them SW1 PM1_Sel, SW2 PM2_Sel

Commit message: input module 1 (controller)
Other:
- title: Module Pip Boy -> Modular Pip Boy
Changed lines of the file:
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@@
 	(paper "A4")
 	(title_block
-		(title "Module Pip Boy")
+		(title "Modular Pip Boy")
 		(rev "1")
 	)
